Commit message: Add 4 wheels to robot

File: src/my_robot/urdf/my_robot.xacro (robot description, xacro)
@@ -14,10 +14,10 @@
     <visual>
       <geometry>
-        <box size="0.4 0.4 0.1"/>
+        <box size="0.5 0.35 0.1"/>
       </geometry>
     </visual>
     <collision>
       <geometry>
-        <box size="0.4 0.4 0.1"/>
+        <box size="0.5 0.3 0.1"/>
       </geometry>
     </collision>
@@ -31,3 +31,131 @@
     </inertial>
   </link>
+  <!-- Create fl wheel -->
+  <link name="wheel_fl">
+    <visual>
+      <origin xyz="0 0 0" rpy=" 0 1.5707 1.5707"/>
+      <geometry>
+        <cylinder radius="0.1" length="0.05"/>
+      </geometry>
+    </visual>
+    <collision>
+      <origin xyz="0 0 0" rpy=" 0 1.5707 1.5707"/>
+      <geometry>
+        <cylinder radius="0.1" length="0.05"/>
+      </geometry>
+    </collision>
+    <inertial>
+      <origin xyz="0 0 0" rpy=" 0 1.5707 1.5707"/>
+      <mass value="5.0"/>
+      <inertia
+          ixx="0.1" ixy="0" ixz="0"
+          iyy="0.1" iyz="0"
+          izz="0.1"
+      />
+    </inertial>
+  </link>
+  <joint type="continuous" name="wheel_fl_hinge">
+    <origin xyz="0.125 0.2 0" rpy="0 0 0"/>
+    <child link="wheel_fl"/>
+    <parent link="chassis"/>
+    <axis xyz="0 1 0" rpy="0 0 0"/>
+    <limit effort="10000" velocity="1000"/>
+    <dynamics damping="1.0" friction="1.0"/>
+  </joint>
+  <!-- Create fr wheel -->
+  <link name="wheel_fr">
+      <visual>
+        <origin xyz="0 0 0" rpy=" 0 1.5707 1.5707"/>
+        <geometry>
+          <cylinder radius="0.1" length="0.05"/>
+        </geometry>
+      </visual>
+      <collision>
+        <origin xyz="0 0 0" rpy=" 0 1.5707 1.5707"/>
+        <geometry>
+          <cylinder radius="0.1" length="0.05"/>
+        </geometry>
+      </collision>
+      <inertial>
+        <origin xyz="0 0 0" rpy=" 0 1.5707 1.5707"/>
+        <mass value="5.0"/>
+        <inertia
+            ixx="0.1" ixy="0" ixz="0"
+            iyy="0.1" iyz="0"
+            izz="0.1"
+        />
+      </inertial>
+    </link>
+    <joint type="continuous" name="wheel_fr_hinge">
+      <origin xyz="0.125 -0.2 0" rpy="0 0 0"/>
+      <child link="wheel_fr"/>
+      <parent link="chassis"/>
+      <axis xyz="0 1 0" rpy="0 0 0"/>
+      <limit effort="10000" velocity="1000"/>
+      <dynamics damping="1.0" friction="1.0"/>
+    </joint>
+    <!-- Create rl wheel -->
+  <link name="wheel_rl">
+      <visual>
+        <origin xyz="0 0 0" rpy=" 0 1.5707 1.5707"/>
+        <geometry>
+          <cylinder radius="0.1" length="0.05"/>
+        </geometry>
+      </visual>
+      <collision>
+        <origin xyz="0 0 0" rpy=" 0 1.5707 1.5707"/>
+        <geometry>
+          <cylinder radius="0.1" length="0.05"/>
+        </geometry>
+      </collision>
+      <inertial>
+        <origin xyz="0 0 0" rpy=" 0 1.5707 1.5707"/>
+        <mass value="5.0"/>
+        <inertia
+            ixx="0.1" ixy="0" ixz="0"
+            iyy="0.1" iyz="0"
+            izz="0.1"
+        />
+      </inertial>
+    </link>
+    <joint type="continuous" name="wheel_rl_hinge">
+      <origin xyz="-0.125 0.2 0" rpy="0 0 0"/>
+      <child link="wheel_rl"/>
+      <parent link="chassis"/>
+      <axis xyz="0 1 0" rpy="0 0 0"/>
+      <limit effort="10000" velocity="1000"/>
+      <dynamics damping="1.0" friction="1.0"/>
+    </joint>
+    <!-- Create rr wheel -->
+  <link name="wheel_rr">
+      <visual>
+        <origin xyz="0 0 0" rpy=" 0 1.5707 1.5707"/>
+        <geometry>
+          <cylinder radius="0.1" length="0.05"/>
+        </geometry>
+      </visual>
+      <collision>
+        <origin xyz="0 0 0" rpy=" 0 1.5707 1.5707"/>
+        <geometry>
+          <cylinder radius="0.1" length="0.05"/>
+        </geometry>
+      </collision>
+      <inertial>
+        <origin xyz="0 0 0" rpy=" 0 1.5707 1.5707"/>
+        <mass value="5.0"/>
+        <inertia
+            ixx="0.1" ixy="0" ixz="0"
+            iyy="0.1" iyz="0"
+            izz="0.1"
+        />
+      </inertial>
+    </link>
+    <joint type="continuous" name="wheel_rr_hinge">
+      <origin xyz="-0.125 -0.2 0" rpy="0 0 0"/>
+      <child link="wheel_rr"/>
+      <parent link="chassis"/>
+      <axis xyz="0 1 0" rpy="0 0 0"/>
+      <limit effort="10000" velocity="1000"/>
+      <dynamics damping="1.0" friction="1.0"/>
+    </joint>
 </robot>

Commit message: Add camera

File: src/my_robot/urdf/my_robot.xacro (robot description, xacro)
@@ -159,3 +159,29 @@
       <dynamics damping="1.0" friction="1.0"/>
     </joint>
+    <!-- Add camera -->
+    <link name="camera">
+      <visual>
+        <geometry>
+          <box size="0.05 0.05 0.05"/>
+        </geometry>
+      </visual>
+      <collision>
+        <geometry>
+          <box size="0.05 0.05 0.05"/>
+        </geometry>
+      </collision>
+      <inertial>
+        <mass value="0.1"/>
+        <inertia
+          ixx="1e-6" ixy="0" ixz="0"
+          iyy="1e-6" iyz="0"
+          izz="1e-6"
+        />
+      </inertial>
+    </link>
+    <joint name="camera_joint" type="fixed">
+      <origin xyz="0.275 0 0.05"/>
+      <parent link="chassis"/>
+      <child link="camera"/>
+    </joint>
 </robot>

Commit message: Add lidar

File: src/my_robot/urdf/my_robot.xacro (robot description, xacro)
@@ -181,7 +181,33 @@
     </link>
     <joint name="camera_joint" type="fixed">
-      <origin xyz="0.275 0 0.05"/>
+      <origin xyz="0.275 0 0" rpy="0 0 0"/>
       <parent link="chassis"/>
       <child link="camera"/>
     </joint>
+    <!-- Add lidar -->
+    <link name = "hokuyo">
+      <visual>
+        <geometry>
+          <mesh filename="package://my_robot/meshes/hokuyo.dae"/>
+        </geometry>
+      </visual>
+      <collision>
+        <geometry>
+          <box size="0.1 0.1 0.1" />
+        </geometry>
+      </collision>
+      <intertial>
+        <mass value="1e-5"/>
+        <inertia
+          ixx="1e-6" ixy="0" ixz="0"
+          iyy="1e-6" iyz="0"
+          izz="1e-6"
+        />
+      </intertial>
+    </link>
+    <joint name="hokuyo_joint" type="fixed">
+      <origin xyz="0.2 0 0.085" rpy="0 0 0"/>
+      <parent link="chassis"/>
+      <child link="hokuyo"/>
+    </joint>
 </robot>

Commit message: Add colors to robot

File: src/my_robot/urdf/my_robot.xacro (robot description, xacro)
@@ -212,3 +212,22 @@
       <child link="hokuyo"/>
     </joint>
+  <!-- Add colors -->
+  <gazebo reference="wheel_fl">
+    <material>Gazebo/Black</material>
+  </gazebo>
+  <gazebo reference="wheel_fr">
+    <material>Gazebo/Black</material>
+  </gazebo>
+  <gazebo reference="wheel_rl">
+    <material>Gazebo/Black</material>
+  </gazebo>
+  <gazebo reference="wheel_rr">
+    <material>Gazebo/Black</material>
+  </gazebo>
+  <gazebo reference="chassis">
+    <material>Gazebo/Brown</material>
+  </gazebo>
+  <gazebo reference="camera">
+    <material>Gazebo/Blue</material>
+  </gazebo>
 </robot>

Commit message: Add skid steer control for 4 wheels

File: src/my_robot/urdf/my_robot.xacro (robot description, xacro)
@@ -226,5 +226,5 @@
   </gazebo>
   <gazebo reference="chassis">
-    <material>Gazebo/Brown</material>
+    <material>Gazebo/Yellow</material>
   </gazebo>
   <gazebo reference="camera">

Commit message: Change wheel dia

File: src/my_robot/urdf/my_robot.xacro (robot description, xacro)
@@ -37,5 +37,5 @@
       <origin xyz="0 0 0" rpy=" 0 1.5707 1.5707"/>
       <geometry>
-        <cylinder radius="0.1" length="0.05"/>
+        <cylinder radius="0.08" length="0.05"/>
       </geometry>
     </visual>
@@ -43,5 +43,5 @@
       <origin xyz="0 0 0" rpy=" 0 1.5707 1.5707"/>
       <geometry>
-        <cylinder radius="0.1" length="0.05"/>
+        <cylinder radius="0.08" length="0.05"/>
       </geometry>
     </collision>
@@ -69,11 +69,11 @@
         <origin xyz="0 0 0" rpy=" 0 1.5707 1.5707"/>
         <geometry>
-          <cylinder radius="0.1" length="0.05"/>
-        </geometry>
-      </visual>
-      <collision>
-        <origin xyz="0 0 0" rpy=" 0 1.5707 1.5707"/>
-        <geometry>
-          <cylinder radius="0.1" length="0.05"/>
+          <cylinder radius="0.08" length="0.05"/>
+        </geometry>
+      </visual>
+      <collision>
+        <origin xyz="0 0 0" rpy=" 0 1.5707 1.5707"/>
+        <geometry>
+          <cylinder radius="0.08" length="0.05"/>
         </geometry>
       </collision>
@@ -101,11 +101,11 @@
         <origin xyz="0 0 0" rpy=" 0 1.5707 1.5707"/>
         <geometry>
-          <cylinder radius="0.1" length="0.05"/>
-        </geometry>
-      </visual>
-      <collision>
-        <origin xyz="0 0 0" rpy=" 0 1.5707 1.5707"/>
-        <geometry>
-          <cylinder radius="0.1" length="0.05"/>
+          <cylinder radius="0.08" length="0.05"/>
+        </geometry>
+      </visual>
+      <collision>
+        <origin xyz="0 0 0" rpy=" 0 1.5707 1.5707"/>
+        <geometry>
+          <cylinder radius="0.08" length="0.05"/>
         </geometry>
       </collision>
@@ -133,11 +133,11 @@
         <origin xyz="0 0 0" rpy=" 0 1.5707 1.5707"/>
         <geometry>
-          <cylinder radius="0.1" length="0.05"/>
-        </geometry>
-      </visual>
-      <collision>
-        <origin xyz="0 0 0" rpy=" 0 1.5707 1.5707"/>
-        <geometry>
-          <cylinder radius="0.1" length="0.05"/>
+          <cylinder radius="0.08" length="0.05"/>
+        </geometry>
+      </visual>
+      <collision>
+        <origin xyz="0 0 0" rpy=" 0 1.5707 1.5707"/>
+        <geometry>
+          <cylinder radius="0.08" length="0.05"/>
         </geometry>
       </collision>
